File: hw/KiCad/STM32WLE5_RF_dongle.kicad_pcb (KiCad board)
At the start: 4 copper layers, 59 x 18 mm, 68 parts, among them J1 Conn_01x02_Pin, J2 cortex-M_debug_connector_10pin, J3 S0941-46R, J4 S0941-46R, J5 S0941-46R, J6 S0941-46R, J7 SMA_142-0701-801_EdgeMount, J8 USB_male_typeA_2.0, T1 DXW21HN5011BL, U1 STM32WLE5C8U6, U2 SKY13453-385LF, U3 USBLC6-2SC6, U4 FT230XS-R, U5 TLV75533PDBVR, Y1 ECS-TXO-25CSMV

Commit message: Fix RF switch VCTL control divider and manufacturing outputs
Parts:
- added G***: LOGO, 1000_user_silk_drawings:RF_Wizard, B.Cu at (123.3, 88.2)
- added R11: 340Ω, 0_resistor_SMD:R_0402_1005Metric, F.Cu at (143.2, 90.2)
- moved C19 2.18 mm to (143.2, 89.2), turned to 0 degrees
- moved R4 0.60 mm to (142.7, 91.7)
Routing:
- net GNDREF: track 167.7 -> 168.8 mm, vias 94 -> 95
- net Net-(U2-VCTL): track 7.28 -> 6.26 mm
